File: TFT_CAN/TFT_CAN.kicad_pcb (KiCad board)
At the start: 2 copper layers, 96.5 x 63.5 mm, 10 parts, among them J1 Conn_01x20, J2 Conn_01x20, J3 Conn_01x06, SW1 Conn_01x02, SW2 Conn_01x02

Commit message: PCBway order
Parts:
- CAN1: moved to B.Cu
- moved CAN1 0.41 mm to (35.3, 81.3), turned to -90 degrees
Routing:
- net GND: track 3.43 -> 0.00 mm, vias 1 -> 0
- net CAN_HI: track 86.3 -> 84.5 mm, vias 1 -> 2
- net CAN_LO: track 88.9 -> 89.7 mm, vias 1 -> 2
- net VBat: track 182.6 -> 183.3 mm, vias 2 -> 3
Other:
- outline, holes or cut-outs redrawn
